File: KiCad/KoalaKeeb/KoalaKeeb.kicad_pcb (KiCad board)
At the start: 2 copper layers, 3.4 x 3 mm, 62 parts, among them J1 JLC_Battery_Con_L, J2 JLC_Battery_Con_R, SW1 Switch_SW_Push, SW10 Switch_SW_Push, SW11 Switch_SW_Push, SW12 Switch_SW_Push, SW13 Switch_SW_Push, SW14 Switch_SW_Push, SW15 Switch_SW_Push, SW16 Switch_SW_Push, SW17 Switch_SW_Push, SW18 Switch_SW_Push, SW19 Switch_SW_Push, SW2 Switch_SW_Push, SW20 Switch_SW_Push, SW21 Switch_SW_Push, SW22 Switch_SW_Push, SW23 Switch_SW_Push, SW24 Switch_SW_Push, SW25 Switch_SW_Push, SW26 Switch_SW_Push, SW27 Switch_SW_Push, SW28 Switch_SW_Push, SW29 Switch_SW_Push, SW3 Switch_SW_Push, SW30 Switch_SW_Push, SW31 Switch_SW_Push, SW32 Switch_SW_Push, SW33 Switch_SW_Push, SW34 Switch_SW_Push, SW4 Switch_SW_Push, SW5 Switch_SW_Push, SW6 Switch_SW_Push, SW7 Switch_SW_Push, SW8 Switch_SW_Push, SW9 Switch_SW_Push, U1 Nice!Nano_L, U2 Nice!Nano_R

Commit message: place all parts for left side
Parts:
- moved L20 395.1 mm to (29.6, 131.2)
- moved L18 394.7 mm to (29.6, 119.3)
- moved L19 394.7 mm to (29.6, 123.6)
- moved L17 394.6 mm to (29.6, 113.5)
- moved L16 394.4 mm to (29.6, 107.6)
- moved L13 384.5 mm to (29.6, 93.9)
- moved L14 384.5 mm to (29.6, 98.2)
- moved L15 384.5 mm to (29.6, 102.6)
- moved L11 384.5 mm to (29.6, 83.7)
- moved L12 384.5 mm to (29.6, 88.1)
- moved power_switch_R1 366.9 mm to (39.0, 23.9)
- moved RSW_R1 352.0 mm to (65.1, 22.0)
- moved J2 327.1 mm to (91.1, 22.0)
- moved power_switch_L1 159.5 mm to (271.0, 82.0), turned to 60 degrees
- moved L10 150.9 mm to (274.0, 71.0)
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
Commit message: place all components on PCB
Parts:
- moved L20 62.5 mm to (46.0, 71.0)
- moved RSW_R1 62.1 mm to (61.0, 84.0), turned to 30 degrees
- moved J2 60.0 mm to (67.1, 77.0), turned to -90 degrees
- moved power_switch_R1 59.0 mm to (49.0, 82.0), turned to -60 degrees
- moved L19 58.0 mm to (46.0, 68.0)
- moved L18 56.7 mm to (46.0, 65.0)
- moved L17 54.0 mm to (46.0, 62.0)
- moved L16 51.3 mm to (46.0, 59.0)
- moved L15 49.4 mm to (46.0, 56.0)
- moved L14 48.1 mm to (46.0, 53.0)
- moved L13 46.9 mm to (46.0, 50.0)
- moved L12 44.2 mm to (46.0, 47.0)
- moved L11 43.0 mm to (46.0, 44.0)
- moved SW32 34.9 mm to (150.0, 83.0)
- moved SW27 34.6 mm to (150.0, 66.0)
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
Commit message: routing and outlines done
Parts:
- moved L11 2.01 mm to (46.2, 42.0)
- moved L1 1.96 mm to (273.9, 42.0)
- moved L12 1.81 mm to (46.2, 45.2)
- moved L2 1.76 mm to (273.9, 45.2)
- moved L13 1.61 mm to (46.2, 48.4)
- moved L3 1.56 mm to (273.9, 48.5)
- moved L14 1.42 mm to (46.2, 51.6)
- moved L4 1.36 mm to (273.9, 51.6)
- moved L15 1.22 mm to (46.2, 54.8)
- moved L5 1.16 mm to (273.9, 54.9)
- moved L16 1.02 mm to (46.2, 58.0)
- moved L6 0.96 mm to (273.9, 58.0)
- moved L17 0.82 mm to (46.2, 61.2)
- moved L7 0.76 mm to (273.9, 61.2)
- moved L18 0.63 mm to (46.2, 64.4)
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Connections:
- U1 pad 10: SW7 -> SW9
- U1 pad 12: SW9 -> SW7
- U1 pad 15: SW15 -> SW11
- U1 pad 16: SW14 -> SW12
- U1 pad 18: SW12 -> SW14
- U1 pad 19: SW11 -> SW15
- U1 pad 2: SW1 -> SW5
- U1 pad 20: SW10 -> SW6
- U1 pad 5: SW2 -> SW4
- U1 pad 7: SW4 -> SW2
- U1 pad 8: SW5 -> SW1
- U1 pad 9: SW6 -> SW10
- U2 pad 10: SW24 -> SW34
- U2 pad 11: SW25 -> SW24
- U2 pad 12: SW26 -> SW33
- U2 pad 13: SW34 -> SW27
- U2 pad 14: SW33 -> SW26
- U2 pad 15: SW32 -> SW25
- U2 pad 16: SW31 -> SW22
- U2 pad 17: SW30 -> SW21
- U2 pad 18: SW29 -> SW20
- U2 pad 19: SW28 -> SW19
- U2 pad 2: SW18 -> SW23
- U2 pad 20: SW27 -> SW18
- U2 pad 5: SW19 -> SW28
- U2 pad 6: SW20 -> SW29
- U2 pad 7: SW21 -> SW30
- U2 pad 8: SW22 -> SW31
- U2 pad 9: SW23 -> SW32
Routing:
- net SW32: track 0.00 -> 114.0 mm
- net SW11: track 0.00 -> 111.0 mm
- net SW6: track 0.00 -> 111.0 mm
- net SW12: track 0.00 -> 110.6 mm
- net SW22: track 0.00 -> 102.9 mm
- net SW13: track 0.00 -> 98.4 mm
- net VCC_R: track 0.00 -> 96.7 mm, vias 0 -> 1
- net SW1: track 0.00 -> 86.9 mm
- net SW27: track 0.00 -> 86.7 mm
- net SW31: track 0.00 -> 85.5 mm
- net SW7: track 0.00 -> 80.9 mm
- net SW14: track 0.00 -> 76.6 mm
- net SW24: track 0.00 -> 75.3 mm, vias 0 -> 1
- net SW2: track 0.00 -> 70.6 mm
- net SW21: track 0.00 -> 70.3 mm
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- added copper zone on B.Cu, net GND_L
- added copper zone on F.Cu, net GND_L
- added copper zone on B.Cu, net GND_R
- added copper zone on F.Cu, net GND_R
Other:
- board size 3.4 x 3 mm -> 236.6 x 86.3 mm
