File: KiCad/KoalaKeeb/KoalaKeeb_v0.2.kicad_pcb (KiCad board)
At the start: 2 copper layers, 238.4 x 86.3 mm, 64 parts, among them J1 JLC_Battery_Con_L, J2 JLC_Battery_Con_R, SW1 Switch_SW_Push, SW10 Switch_SW_Push, SW11 Switch_SW_Push, SW12 Switch_SW_Push, SW13 Switch_SW_Push, SW14 Switch_SW_Push, SW15 Switch_SW_Push, SW16 Switch_SW_Push, SW17 Switch_SW_Push, SW18 Switch_SW_Push, SW19 Switch_SW_Push, SW2 Switch_SW_Push, SW20 Switch_SW_Push, SW21 Switch_SW_Push, SW22 Switch_SW_Push, SW23 Switch_SW_Push, SW24 Switch_SW_Push, SW25 Switch_SW_Push, SW26 Switch_SW_Push, SW27 Switch_SW_Push, SW28 Switch_SW_Push, SW29 Switch_SW_Push, SW3 Switch_SW_Push, SW30 Switch_SW_Push, SW31 Switch_SW_Push, SW32 Switch_SW_Push, SW33 Switch_SW_Push, SW34 Switch_SW_Push, SW4 Switch_SW_Push, SW5 Switch_SW_Push, SW6 Switch_SW_Push, SW7 Switch_SW_Push, SW8 Switch_SW_Push, SW9 Switch_SW_Push, U1 Nice!Nano_L, U2 Nice!Nano_R

Commit message: add v0.2
Parts:
- moved L1 2.15 mm to (276.0, 42.0)
- moved L10 2.15 mm to (276.0, 70.8), turned to 180 degrees
- moved L2 2.15 mm to (276.0, 45.2), turned to 180 degrees
- moved L3 2.15 mm to (276.0, 48.5)
- moved L4 2.15 mm to (276.0, 51.6), turned to 180 degrees
- moved L5 2.15 mm to (276.0, 54.9)
- moved L6 2.15 mm to (276.0, 58.0), turned to 180 degrees
- moved L7 2.15 mm to (276.0, 61.2)
- moved L8 2.15 mm to (276.0, 64.5), turned to 180 degrees
- moved L9 2.15 mm to (276.0, 67.7)
- moved U1 1.00 mm to (261.0, 57.0)
- moved power_switch_L1 0.55 mm to (271.3, 82.5), turned to 59 degrees
- moved power_switch_R1 0.55 mm to (48.8, 82.5), turned to -59 degrees
Routing:
- net SW6: track 0.00 -> 113.1 mm
- net SW11: track 0.00 -> 104.7 mm
- net SW12: track 0.00 -> 103.6 mm
- net SW13: track 0.00 -> 89.0 mm
- net SW1: track 0.00 -> 88.5 mm
- net SW2: track 0.00 -> 84.7 mm
- net SW7: track 0.00 -> 82.5 mm
- net VCC_L: track 0.00 -> 76.6 mm, vias 0 -> 6
- net SW14: track 0.00 -> 70.6 mm
- net SW8: track 0.00 -> 69.2 mm
- net SW3: track 0.00 -> 65.9 mm
- net SW16: track 0.00 -> 58.4 mm
- net SW15: track 0.00 -> 57.2 mm
- net SW4: track 0.00 -> 44.8 mm
- net RST_L: track 0.00 -> 44.7 mm, vias 0 -> 2
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- added copper zone on B.Cu, net GND_L
- added copper zone on F.Cu, net GND_L
- added copper zone on B.Cu, net GND_R
- added copper zone on F.Cu, net GND_R
Other:
- board size 238.4 x 86.3 mm -> 240.9 x 86.3 mm
